Commit message: sensor simulation.

File: description/boties.urdf (robot description, URDF)
Before this commit: robot boties, 5 links, 4 joints
Links:
- removed link leftWheel_link
- removed link rightWheel_link
- added link camera_link; collision box size=0.02 0.05 0.02; visual box size=0.02 0.05 0.02
- added link left_wheel, mass 10; collision cylinder length=0.05 radius=0.05; visual cylinder length=0.05 radius=0.05
- added link right_wheel, mass 10; collision cylinder length=0.05 radius=0.05; visual cylinder length=0.05 radius=0.05
- link base_link: geometry collision cylinder length=0.08 radius=0.1; visual cylinder length=0.08 radius=0.1
Joints:
- added joint camera_joint: type fixed, parent base_link, child camera_link, origin xyz=0 0.05 0.05 rpy=0 0 1.57075, axis 0 1 0
- joint baseToLeftWheel_joint: child leftWheel_link -> left_wheel
- joint baseToRightWheel_joint: child rightWheel_link -> right_wheel
